File: Electronics v0.2.1/kicad/gamegirl-v02.sch (KiCad schematic (older format))
At the start: 93 parts, among them P1 Molex 47346-0001, P2 PI-ZERO, Q1 Q_NMOS_DGS, Q2 DMC2020, Q3 Q_PMOS_DGS, Q4 Q_PMOS_DGS, SW1 JSX08001SAQNL, SW10 Y, SW11 X, SW12 B, SW13 A, SW2 UP, SW3 DOWN, SW4 RIGHT, SW5 LEFT, SW6 STA, SW7 SEL, SW8 L1, SW9 R1, U1 ER-TFT024-3, U2 ETA9740, U3 PAM8302A, U4 RTL8188, U5 MCP23S17, U6 ADCMP354, U7 LP5907

Commit message: Update gamegirl-v02.sch
Parts:
- AE1: symbol Antenna_Shield -> Device:Antenna_Shield
- C1, C10, C12, C13, C14, C15, C16, C17, C18, C19, C2, C20, C21, C22, C23, C24, C25, C26, C3, C4, C5, C6, C7, C8, C9: symbol C -> Device:C
- C11: symbol CP -> Device:CP
- D3: symbol D_Schottky_x2_KCom_AAK -> Device:D_Schottky_x2_KCom_AAK
- JP1: symbol Jumper_NC_Dual -> Device:Jumper_NC_Dual
- JP2: symbol Jumper_NC_Small -> Device:Jumper_NC_Small
- JP3: symbol Jumper_USB_90ohm -> gamegirl-v02:Jumper_USB_90ohm
- L1, R1, R10, R11, R12, R13, R14, R15, R16, R17, R18, R19, R2, R20, R21, R22, R23, R24, R27, R3, R4, R5, R6, R7, R8, R9: symbol R -> Device:R
- L2: symbol L_Small -> Device:L_Small
- P2: symbol PI-ZERO -> gamegirl-v02:PI-ZERO
- Q1: symbol Q_NMOS_GSD -> Device:Q_NMOS_GSD
- Q3, Q4: symbol Q_PMOS_GSD -> Device:Q_PMOS_GSD
- SP1: symbol SPEAKER -> Device:Speaker
- U1: symbol ER-TFT024-3 -> gamegirl-v02:ER-TFT024-3
- U2: symbol ETA9740 -> gamegirl-v02:ETA9740
- U3: symbol PAM8302A -> gamegirl-v02:PAM8302A
- U4: symbol RTL8188 -> gamegirl-v02:RTL8188
- U7: symbol LP5907 -> gamegirl-v02:LP5907
Connections:
- wire segments 227 -> 282
